File: Current Driver/Current Driver_V3.kicad_sch (KiCad schematic)
At the start: 64 parts, among them J1 VP BJT Conn, J2 VN BJT Conn, J3 Load, J4 Input, J5 PWR In, J6 Add. R, Q1 D45H11, Q2 D45H11G, Q3 BC817, Q4 BC807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

Commit message: PCB V3
Parts:
- added H1, H2, H3, H4: MountingHole_Pad, MountingHole:MountingHole_3.2mm_M3_DIN965_Pad_TopBottom, symbol Mechanical:MountingHole_Pad
Connections:
- net GND: now also H1.1, H2.1, H3.1, H4.1
