File: Current Driver/Current Driver_V3.kicad_pcb (KiCad board)
At the start: 2 copper layers, 70 x 70 mm, 68 parts, among them J1 VP BJT Conn, J2 VN BJT Conn, J3 Load, J4 Input, J5 PWR In, J6 Add. R, Q1 D45H11, Q2 D45H11G, Q3 BC817, Q4 BC807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

Commit message: Update PCB
Parts:
- moved R15 20.3 mm to (192.0, 102.2)
- moved R36 20.1 mm to (191.9, 111.5)
- moved C9 19.5 mm to (186.5, 134.5), turned to 90 degrees
- moved R19 17.8 mm to (170.2, 121.0)
- moved C8 16.9 mm to (179.0, 134.5), turned to 90 degrees
- moved R22 16.4 mm to (172.2, 125.0)
- moved R5 15.6 mm to (164.5, 121.0)
- moved R23 14.9 mm to (174.8, 125.0)
- moved R2 14.8 mm to (162.5, 125.0)
- moved R3 14.0 mm to (160.0, 125.0)
- moved D2 13.8 mm to (170.2, 124.5), turned to -90 degrees
- moved C10 13.7 mm to (157.0, 134.5), turned to -90 degrees
- moved Q6 12.5 mm to (188.2, 122.7), turned to 90 degrees
- moved D1 12.0 mm to (164.5, 124.5), turned to 90 degrees
- moved TP1 12.0 mm to (146.2, 92.8)
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Routing:
- net /DRIVING_OUTPUT: track 62.7 -> 0.00 mm
- net GND: track 42.6 -> 2.83 mm, vias 19 -> 42
- net +VCC: track 174.7 -> 138.8 mm
- net /DRIVING_INPUT: track 70.8 -> 48.6 mm, vias 4 -> 2
- net /VNEG_B: track 52.9 -> 34.9 mm, vias 0 -> 1
- net Net-(Q2-C): track 23.4 -> 30.7 mm
- net /VPOS_B: track 36.7 -> 29.7 mm
- net -VCC: track 129.2 -> 136.0 mm, vias 2 -> 3
- net /V_REF: track 14.7 -> 21.2 mm
- net Net-(Q4-E): track 19.6 -> 25.9 mm
- net +3.3V: track 10.3 -> 16.0 mm
- net /VNEG_C: track 14.1 -> 11.7 mm
- net Net-(Q3-B): track 5.56 -> 3.37 mm
- net /VPOS_C: track 14.6 -> 13.1 mm
- net Net-(D1-A): track 5.19 -> 3.88 mm
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- added copper zone on F.Cu, net /DRIVING_OUTPUT
- added copper zone on F.Cu, net GND
